Commit message: u

File: mani_skill2_real2sim/assets/descriptions/rm65b_description/rm_65_b_description.urdf (robot description, URDF)
Before this commit: robot rm_65_b, 15 links, 14 joints
Links:
- link 4C2_Link1: geometry collision mesh filename=meshes/4C2_Link1.STL; visual mesh filename=meshes/4C2_Link1.STL
- link 4C2_Link2: geometry collision mesh filename=meshes/4C2_Link2.STL; visual mesh filename=meshes/4C2_Link2.STL
- link 4C2_Link3: geometry collision mesh filename=meshes/4C2_Link3.STL; visual mesh filename=meshes/4C2_Link3.STL
- link 4C2_Link4: geometry collision mesh filename=meshes/4C2_Link4.STL; visual mesh filename=meshes/4C2_Link4.STL
- link 4C2_Link5: geometry collision mesh filename=meshes/4C2_Link5.STL; visual mesh filename=meshes/4C2_Link5.STL
- link 4C2_Link6: geometry collision mesh filename=meshes/4C2_Link6.STL; visual mesh filename=meshes/4C2_Link6.STL
- link 4C2_baselink: geometry collision mesh filename=meshes/4C2_baselink.STL; visual mesh filename=meshes/4C2_baselink.STL
- link Link1: geometry collision mesh filename=meshes/link1.STL; visual mesh filename=meshes/link1.STL
- link Link2: geometry collision mesh filename=meshes/link2.STL; visual mesh filename=meshes/link2.STL
- link Link3: geometry collision mesh filename=meshes/link3.STL; visual mesh filename=meshes/link3.STL
- link Link4: geometry collision mesh filename=meshes/link4.STL; visual mesh filename=meshes/link4.STL
- link Link5: geometry collision mesh filename=meshes/link5.STL; visual mesh filename=meshes/link5.STL
- link Link6: geometry collision mesh filename=meshes/link6.STL; visual mesh filename=meshes/link6.STL
- link base_link: geometry collision mesh filename=meshes/base_link.STL; visual mesh filename=meshes/base_link.STL
- link fixed_plate_link: geometry collision mesh filename=meshes/fixed_plate.STL; visual mesh filename=meshes/fixed_plate.STL
Joints:
- removed joint gripper_base_link
- added joint gripper_base: type fixed, parent Link6, child 4C2_baselink
- joint fixed_plate: axis 0 0 1 -> (none); origin xyz=0 0 0.057 rpy=3.1415 0 0 -> xyz=0 0 -0.052 rpy=0 0 0
